File: kicad/default/mrc_template.kicad_sch (KiCad schematic)
At the start: 0 parts

Commit message: readme
Other:
- title: <<PROJECT TITLE>> -> ${MRC_TITLE}
Changed lines of the file:
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@@
 	(paper "A4")
 	(title_block
-		(title "<<PROJECT TITLE>>")
-		(date "MM/DD/YYYY")
-		(rev "<<XX.XX>>")
+		(title "${MRC_TITLE}")
+		(date "${MRC_DATE}")
+		(rev "${MRC_REVISION}")
 		(company "BU Mars Rover Club Electrical Team")
-		(comment 1 "<<DESCRIPTION LINE 2>>")
-		(comment 2 "<<DESCRIPTION LINE 1>>")
-		(comment 3 "<<CONTRIBUTORS>>")
-		(comment 4 "<<SUBSYSTEM>>")
+		(comment 1 "${MRC_DESC_2}")
+		(comment 2 "${MRC_DESC_1}")
+		(comment 3 "${MRC_CONTRIBUTORS}")
+		(comment 4 "${MRC_SUBSYSTEM}")
 	)
 	(sheet_instances
